File: henryfc_v1.1.sch (EAGLE design)
At the start: 59 parts, among them IC2 ICM-20602, IC3 AT7456E, IC4 STM32F722RET6TR, J2 10118192-0001LF, X1 SM07B-SRSS-TB, Y1 NX3225GA-27.000M-STD-CRG-1, Y2 ECS-80-12-33-JGN-TR

Commit message: update 5v reg
Parts:
- removed Y2: ECS-80-12-33-JGN-TR, SamacSys_Parts:ECS-80-12-33-JGN-TR
- added C3, C6: 0.1uF, rcl:C-EUC0805
- added C4, C7: 10uF, rcl:C-EUC0805
- added IC1, IC5: LM317DCYR, SamacSys_Parts:LM317DCYR
- added PAD10: BOOT, wirepad:SMD2
- added R12, R3: 1k, rcl:R-EU_R0603
- added R2, R4: 3k, rcl:R-EU_R0603
- C19: value 4.7uF -> 2.2uF
- R1: value 10K -> CSTCE8M00G55-R0; device rcl:R-EU_R0603 -> SamacSys_Parts:CSTCE8M00G55-R0
- X1: device con-JST:SM07B-SRSS-TB -> con-jst:SM07B-SRSS-TB
Connections:
- removed net LED0: IC4.PB9, R9.1
- removed net N$3: PAD3.P, R1.2
- new net 5V_REG1: IC5.OUTPUT_1, IC5.OUTPUT_2, R3.2
- new net N$1: IC5.ADJUST, R2.2, R3.1
- new net N$2: IC1.ADJUST, R12.1, R4.2
- net 3.3V_REG: now also PAD10.P, R9.1
- net 5V_REG: now also IC1.OUTPUT_1, IC1.OUTPUT_2, R12.2
- net BOOT: now also PAD3.P, R11.1; no longer R1.1, R11.2
- net GND: now also C24.1, C3.1, C4.1, C6.1, C7.1, R1.2, R11.2, R2.1, R4.1; no longer C24.2, R11.1, Y2.GND_1, Y2.GND_2
- net NRST: now also C24.2; no longer C24.1
- net OSC_IN: now also R1.1; no longer Y2.OUT/IN
- net OSC_OUT: now also R1.3; no longer Y2.IN/OUT
- net VCC: now also C3.2, C4.2, C6.2, C7.2, IC1.INPUT, IC5.INPUT
Other:
- moved on the sheet: C24, R11

Commit message: update PCB layout
Parts:
- removed PAD10: BOOT, wirepad:SMD2
- added C26: 10uF, rcl:C-EUC0805
- added C8: 0.1uF, rcl:C-EUC0805
Connections:
- net +5V: now also C26.2, C8.2; no longer PAD19.P, PAD20.P
- net 3.3V_REG: no longer PAD10.P
- net 5V_REG1: now also PAD19.P, PAD20.P
- net GND: now also C26.1, C8.1
Changed lines of the file:
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@@
 <part name="SUPPLY5" library="supply2" library_urn="urn:adsk.eagle:library:372" deviceset="GND" device=""/>
 <part name="SUPPLY6" library="supply2" library_urn="urn:adsk.eagle:library:372" deviceset="GND" device=""/>
-<part name="PAD10" library="wirepad" library_urn="urn:adsk.eagle:library:412" deviceset="SMD2" device="" package3d_urn="urn:adsk.eagle:package:30839/1" value="BOOT"/>
 <part name="R1" library="SamacSys_Parts" deviceset="CSTCE8M00G55-R0" device=""/>
 <part name="SUPPLY7" library="supply2" library_urn="urn:adsk.eagle:library:372" deviceset="GND" device=""/>
@@
 <part name="SUPPLY28" library="supply2" library_urn="urn:adsk.eagle:library:372" deviceset="GND" device=""/>
 <part name="SUPPLY29" library="supply2" library_urn="urn:adsk.eagle:library:372" deviceset="GND" device=""/>
+<part name="C8" library="rcl" library_urn="urn:adsk.eagle:library:334" deviceset="C-EU" device="C0805" package3d_urn="urn:adsk.eagle:package:23617/2" value="0.1uF"/>
+<part name="SUPPLY30" library="supply2" library_urn="urn:adsk.eagle:library:372" deviceset="GND" device=""/>
+<part name="C26" library="rcl" library_urn="urn:adsk.eagle:library:334" deviceset="C-EU" device="C0805" package3d_urn="urn:adsk.eagle:package:23617/2" value="10uF"/>
+<part name="SUPPLY31" library="supply2" library_urn="urn:adsk.eagle:library:372" deviceset="GND" device=""/>
 </parts>
 <sheets>
@@
 <attribute name="VALUE" x="-116.205" y="-13.335" size="1.778" layer="96"/>
 </instance>
-<instance part="PAD10" gate="1" x="-50.8" y="55.88" smashed="yes">
-<attribute name="NAME" x="-51.943" y="57.7342" size="1.778" layer="95"/>
-<attribute name="VALUE" x="-51.943" y="52.578" size="1.778" layer="96"/>
-</instance>
 <instance part="R1" gate="G$1" x="-147.32" y="10.16" smashed="yes">
 <attribute name="NAME" x="-130.81" y="17.78" size="1.778" layer="95" align="center-left"/>
@@
 <instance part="SUPPLY29" gate="GND" x="10.16" y="38.1" smashed="yes">
 <attribute name="VALUE" x="9.525" y="34.925" size="1.778" layer="96"/>
+</instance>
+<instance part="C8" gate="G$1" x="-187.96" y="68.58" smashed="yes" rot="R180">
+<attribute name="NAME" x="-189.484" y="68.199" size="1.778" layer="95" rot="R180"/>
+<attribute name="VALUE" x="-189.484" y="73.279" size="1.778" layer="96" rot="R180"/>
+</instance>
+<instance part="SUPPLY30" gate="GND" x="-187.96" y="63.5" smashed="yes">
+<attribute name="VALUE" x="-188.595" y="60.325" size="1.778" layer="96"/>
+</instance>
+<instance part="C26" gate="G$1" x="-177.8" y="68.58" smashed="yes" rot="R180">
+<attribute name="NAME" x="-179.324" y="68.199" size="1.778" layer="95" rot="R180"/>
+<attribute name="VALUE" x="-179.324" y="73.279" size="1.778" layer="96" rot="R180"/>
+</instance>
+<instance part="SUPPLY31" gate="GND" x="-177.8" y="63.5" smashed="yes">
+<attribute name="VALUE" x="-178.435" y="60.325" size="1.778" layer="96"/>
 </instance>
 </instances>
@@
 <segment>
 <pinref part="D1" gate="G$1" pin="CATHODE"/>
-<wire x1="-190.5" y1="78.74" x2="-182.88" y2="78.74" width="0.1524" layer="91"/>
-<label x="-182.88" y="78.74" size="1.778" layer="95"/>
+<wire x1="-190.5" y1="78.74" x2="-187.96" y2="78.74" width="0.1524" layer="91"/>
+<label x="-175.26" y="78.74" size="1.778" layer="95"/>
+<pinref part="C8" gate="G$1" pin="2"/>
+<wire x1="-187.96" y1="78.74" x2="-177.8" y2="78.74" width="0.1524" layer="91"/>
+<wire x1="-177.8" y1="78.74" x2="-175.26" y2="78.74" width="0.1524" layer="91"/>
+<wire x1="-187.96" y1="73.66" x2="-187.96" y2="78.74" width="0.1524" layer="91"/>
+<junction x="-187.96" y="78.74"/>
+<pinref part="C26" gate="G$1" pin="2"/>
+<wire x1="-177.8" y1="73.66" x2="-177.8" y2="78.74" width="0.1524" layer="91"/>
+<junction x="-177.8" y="78.74"/>
 </segment>
 <segment>
@@
 <junction x="43.18" y="-35.56"/>
 <label x="38.1" y="-35.56" size="1.778" layer="95"/>
-</segment>
-<segment>
-<pinref part="PAD20" gate="1" pin="P"/>
-<wire x1="-165.1" y1="83.82" x2="-162.56" y2="83.82" width="0.1524" layer="91"/>
-<label x="-160.02" y="83.82" size="1.778" layer="95"/>
-</segment>
-<segment>
-<pinref part="PAD19" gate="1" pin="P"/>
-<wire x1="-165.1" y1="76.2" x2="-162.56" y2="76.2" width="0.1524" layer="91"/>
-<label x="-160.02" y="76.2" size="1.778" layer="95"/>
 </segment>
 <segment>
@@
 <pinref part="SUPPLY29" gate="GND" pin="GND"/>
 </segment>
+<segment>
+<pinref part="C8" gate="G$1" pin="1"/>
+<pinref part="SUPPLY30" gate="GND" pin="GND"/>
+</segment>
+<segment>
+<pinref part="SUPPLY31" gate="GND" pin="GND"/>
+<pinref part="C26" gate="G$1" pin="1"/>
+</segment>
 </net>
 <net name="VCC" class="0">
@@
 <wire x1="-27.94" y1="15.24" x2="-22.86" y2="15.24" width="0.1524" layer="91"/>
 <label x="-22.86" y="15.24" size="1.778" layer="95"/>
-</segment>
-<segment>
-<pinref part="PAD10" gate="1" pin="P"/>
-<wire x1="-48.26" y1="55.88" x2="-40.64" y2="55.88" width="0.1524" layer="91"/>
-<label x="-38.1" y="55.88" size="1.778" layer="95"/>
 </segment>
 <segment>
@@
 <label x="48.26" y="2.54" size="1.778" layer="95" rot="R180"/>
 </segment>
-</net>
+<segment>
+<pinref part="PAD20" gate="1" pin="P"/>
+<wire x1="-165.1" y1="83.82" x2="-162.56" y2="83.82" width="0.1524" layer="91"/>
+<label x="-160.02" y="83.82" size="1.778" layer="95"/>
+</segment>
+<segment>
+<pinref part="PAD19" gate="1" pin="P"/>
+<wire x1="-165.1" y1="76.2" x2="-162.56" y2="76.2" width="0.1524" layer="91"/>
+<label x="-160.02" y="76.2" size="1.778" layer="95"/>
+</segment>
+</net>

Commit message: finalized PCB
Parts:
- PAD8: value LED_STRIP -> LED
Changed lines of the file:
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@@
 <part name="PAD6" library="wirepad" library_urn="urn:adsk.eagle:library:412" deviceset="SMD2" device="" package3d_urn="urn:adsk.eagle:package:30839/1" value="RX3"/>
 <part name="PAD7" library="wirepad" library_urn="urn:adsk.eagle:library:412" deviceset="SMD2" device="" package3d_urn="urn:adsk.eagle:package:30839/1" value="TX3"/>
-<part name="PAD8" library="wirepad" library_urn="urn:adsk.eagle:library:412" deviceset="SMD2" device="" package3d_urn="urn:adsk.eagle:package:30839/1" value="LED_STRIP"/>
+<part name="PAD8" library="wirepad" library_urn="urn:adsk.eagle:library:412" deviceset="SMD2" device="" package3d_urn="urn:adsk.eagle:package:30839/1" value="LED"/>
 <part name="PAD9" library="wirepad" library_urn="urn:adsk.eagle:library:412" deviceset="SMD2" device="" package3d_urn="urn:adsk.eagle:package:30839/1" value="GND"/>
 <part name="PAD11" library="wirepad" library_urn="urn:adsk.eagle:library:412" deviceset="SMD2" device="" package3d_urn="urn:adsk.eagle:package:30839/1" value="TX1"/>

Commit message: cleaned files
Other:
- note added: "DATE: 21/10/2020"
- note added: "REV: 1.1"
- note removed: "DATE: 24/07/2020"
- note removed: "REV: 1.0"
Changed lines of the file:
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@@
 <frame x1="-264.16" y1="-104.14" x2="139.7" y2="157.48" columns="8" rows="5" layer="91"/>
 <text x="78.74" y="-88.9" size="1.778" layer="91">TITLE:    HENRYFC</text>
-<text x="119.38" y="-88.9" size="1.778" layer="91">REV:    1.0</text>
+<text x="119.38" y="-88.9" size="1.778" layer="91">REV:    1.1</text>
 <text x="81.28" y="-96.52" size="1.778" layer="91">SHEET:   1/1</text>
-<text x="114.3" y="-96.52" size="1.778" layer="91">DATE:    24/07/2020</text>
+<text x="111.76" y="-96.52" size="1.778" layer="91">DATE:    21/10/2020</text>
 </plain>
 <instances>
