File: henryfc v2.sch (EAGLE design)
At the start: 97 parts, among them X1 SM07B-SRSS-TB

Commit message: cleaning up schematic
Connections:
- removed net GYRO_1_CS_PIN: U$8.CS
- removed net GYRO_1_EXTI_PIN: U$8.INT
- removed net N$17: U$5.PB12
- removed net N$22: U$5.PC1
- net GYRO1_CS_PIN: now also U$8.CS
- net GYRO1_EXTI_PIN: now also U$8.INT
Other:
- moved on the sheet: C1, C10, C11, C12, C13, C14, C15, C16, C17, C18, C19, C2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
