File: henryfc v2.brd (EAGLE design)
At the start: 30 x 30 mm, 74 parts, among them X1 SM07B-SRSS-TB

Commit message: more pcb work
Parts:
- moved R10 4.10 mm to (20.8, 9.50)
- moved R9 4.00 mm to (16.8, 9.50)
- moved C9 3.70 mm to (2.70, 20.1), turned to 270 degrees
- moved C7 3.42 mm to (1.70, 22.9), turned to 90 degrees
- moved C8 3.00 mm to (4.70, 20.1), turned to 180 degrees
- moved C13 2.02 mm to (4.40, 16.7)
- moved C14 1.66 mm to (4.40, 17.9), turned to 0 degrees
- moved C10 1.62 mm to (1.50, 20.1)
- moved LED1 1.60 mm to (19.6, 9.50)
- moved LED2 1.60 mm to (18.0, 9.50)
- moved U$8 1.32 mm to (4.10, 23.0), turned to 180 degrees
- moved R8 0.22 mm to (15.0, 8.00), turned to 180 degrees
- moved R11 0.22 mm to (15.0, 9.20)
- moved C16 0.20 mm to (9.30, 28.9)
- moved C1 0.14 mm to (23.2, 5.10)
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Routing:
- net 3V3: track 0.00 -> 79.9 mm, vias 0 -> 5
- net VCC: track 0.00 -> 24.9 mm, vias 0 -> 2
- net 5V: track 0.00 -> 10.3 mm, vias 0 -> 2
- net SPI1_SCK_PIN: track 0.00 -> 6.64 mm, vias 0 -> 2
- net 5V_USB: track 0.00 -> 5.49 mm
- net 5V_REG-A: track 0.00 -> 5.37 mm
- net GND: track 0.00 -> 2.69 mm
- net N$10: track 0.00 -> 2.25 mm
- net SPI1_MOSI_PIN: track 0.00 -> 2.01 mm
- net SPI1_MISO_PIN: track 0.00 -> 2.01 mm
